Commit message: Finished robot model, added camera topic

File: mybot_description/urdf/macros.xacro (robot description, xacro)
@@ -38,5 +38,5 @@
             <parent link="chassis"/>
             <child link="${lr}_rear_wheel"/>
-            <origin xyz="${-wheelPos+chassisLength/2} ${tY*wheelWidth/2+tY*chassisWidth/2} ${wheelRadius}" rpy="0 0 0" />
+            <origin xyz="${-wheelPos+chassisLength/2} ${tY*wheelWidth/2+tY*0.01+tY*chassisWidth/2} ${wheelRadius}" rpy="0 0 0" />
             <axis xyz="0 1 0" rpy="0 0 0" />
             <limit effort="100" velocity="100"/>
@@ -50,5 +50,5 @@
             <actuator name="${lr}_rear_Motor">
                 <mechanicalReduction>10</mechanicalReduction>
-                <hardwareInterface>hardware_interface/EffortJointInterface</hardwareInterface>
+                <hardwareInterface>hardware_interface/VelocityJointInterface</hardwareInterface>
             </actuator>
         </transmission>
@@ -80,5 +80,5 @@
             <kp value="10000000.0" />
             <kd value="1.0" />
-            <fdir1 value="0 0 1"/>
+            <fdir1 value="0 0 0"/>
             <material>Gazebo/Black</material>
         </gazebo>
@@ -87,11 +87,11 @@
                 <origin xyz="0 0 0" rpy="0 0 0" />
                 <geometry>
-                    <box size="0.001 0.001 0.001" />
+                    <box size="0.06 0.06 0.06" />
                 </geometry>
             </visual>
             <inertial>
                 <origin xyz="0 0 0" rpy="0 0 0" />
-                <mass value="${wheelMass}"/>
-                <box_inertia m="1" x="0.001" y="0.001" z="0.001"/>
+                <mass value="1"/>
+                <box_inertia m="1" x="0.06" y="0.06" z="0.06"/>
             </inertial>
         </link>
@@ -100,5 +100,5 @@
         </gazebo>
         <joint name="${lr}_steer_joint" type="revolute">
-            <origin xyz="${wheelPos-chassisLength/2}  ${tY*wheelWidth/2+tY*chassisWidth/2}  ${wheelRadius}" rpy="0.0 0.0 0.0"/>
+            <origin xyz="${wheelPos-chassisLength/2}  ${tY*wheelWidth/2+tY*0.01+tY*chassisWidth/2}  ${wheelRadius}" rpy="0.0 0.0 0.0"/>
             <parent link="chassis"/>
             <child link="${lr}_steer"/>

File: mybot_description/urdf/mybot.xacro (robot description, xacro)
@@ -4,5 +4,5 @@
     <xacro:property name="PI" value="3.1415926535897931"/>
     <xacro:property name="chassisHeight" value="0.1"/>
-    <xacro:property name="chassisLength" value="0.4"/>
+    <xacro:property name="chassisLength" value="0.6"/>
     <xacro:property name="chassisWidth" value="0.2"/>
     <xacro:property name="chassisMass" value="50"/>
@@ -11,5 +11,5 @@
     <xacro:property name="wheelWidth" value="0.05"/>
     <xacro:property name="wheelRadius" value="0.08"/>
-    <xacro:property name="wheelPos" value="0.3"/>
+    <xacro:property name="wheelPos" value="0.45"/>
     <xacro:property name="wheelMass" value="5"/>
     <xacro:property name="cameraSize" value="0.05"/>
@@ -47,3 +47,28 @@
     <front_wheel lr="right" tY="-1" />
     <front_wheel lr="left" tY="1" />
+    <link name="camera">
+        <collision>
+            <origin xyz="0 0 0" rpy="0 0 0"/>
+            <geometry>
+                <box size="${cameraSize} ${cameraSize} ${cameraSize}"/>
+            </geometry>
+        </collision>
+        <visual>
+            <origin xyz="0 0 0" rpy="0 0 0"/>
+            <geometry>
+                <box size="${cameraSize} ${cameraSize} ${cameraSize}"/>
+            </geometry>
+            <material name="blue"/>
+        </visual>
+        <inertial>
+            <mass value="${cameraMass}" />
+            <origin xyz="0 0 0" rpy="0 0 0"/>
+            <box_inertia m="${cameraMass}" x="${cameraSize}" y="${cameraSize}" z="${cameraSize}" />
+        </inertial>
+    </link>
+    <joint name="camera_joint" type="fixed">
+        <origin xyz="${chassisLength/2} 0.0 ${chassisHeight}" rpy="0.0 0.0 0.0"/>
+        <parent link="chassis"/>
+        <child link="camera"/>
+    </joint>
 </robot>

Commit message: working velocity controller and laser addition

File: mybot_description/urdf/macros.xacro (robot description, xacro)
@@ -2,4 +2,5 @@
 <robot name="mybot"
     xmlns:xacro="http://www.ros.org/wiki/xacro">
+    <!-- PARAMETERS SETTINGS: INERTIA OF ALL KIND OF GEOMETRY OBJECT -->
     <macro name="cylinder_inertia" params="m r h">
         <inertia ixx="${m*(3*r*r+h*h)/12}" ixy = "0" ixz = "0" iyy="${m*(3*r*r+h*h)/12}" iyz = "0" izz="${m*r*r/2}" />
@@ -11,4 +12,5 @@
         <inertia ixx="${2*m*r*r/5}" ixy = "0" ixz = "0" iyy="${2*m*r*r/5}" iyz = "0" izz="${2*m*r*r/5}" />
     </macro>
+    <!-- REAR WHEEL MACROS -->
     <macro name="rear_wheel" params="lr tY">
         <link name="${lr}_rear_wheel">
@@ -46,5 +48,5 @@
             <type>transmission_interface/SimpleTransmission</type>
             <joint name="${lr}_rear_wheel_hinge">
-                <hardwareInterface>hardware_interface/EffortJointInterface</hardwareInterface>
+                <hardwareInterface>hardware_interface/VelocityJointInterface</hardwareInterface>
             </joint>
             <actuator name="${lr}_rear_Motor">
@@ -54,4 +56,5 @@
         </transmission>
     </macro>
+    <!-- FRONT WHEEL MACRO -->
     <macro name="front_wheel" params="lr tY">
         <link name="${lr}_front_wheel">
@@ -76,9 +79,4 @@
         </link>
         <gazebo reference="${lr}_front_wheel">
-            <mu1 value="1.0"/>
-            <mu2 value="1.0"/>
-            <kp value="10000000.0" />
-            <kd value="1.0" />
-            <fdir1 value="0 0 0"/>
             <material>Gazebo/Black</material>
         </gazebo>
@@ -116,5 +114,5 @@
             <type>transmission_interface/SimpleTransmission</type>
             <joint name="${lr}_steer_joint">
-                <hardwareInterface>hardware_interface/EffortJointInterface </hardwareInterface>
+                <hardwareInterface>hardware_interface/PositionJointInterface </hardwareInterface>
             </joint>
             <actuator name="${lr}_front_Motor">
@@ -124,4 +122,5 @@
         </transmission>
     </macro>
+    <!-- CASTOR WHEELS MACRO -->
     <macro name="front_castor_wheel">
         <joint name="fixed" type="fixed">

File: mybot_description/urdf/mybot.xacro (robot description, xacro)
@@ -68,7 +68,26 @@
     </link>
     <joint name="camera_joint" type="fixed">
-        <origin xyz="${chassisLength/2} 0.0 ${chassisHeight}" rpy="0.0 0.0 0.0"/>
+        <origin xyz="${chassisLength/2} 0 ${chassisHeight}" rpy="0.0 0.0 0.0"/>
         <parent link="chassis"/>
         <child link="camera"/>
     </joint>
+    <link name="base_laser_link">
+        <visual>
+            <origin xyz="0 0 0" rpy="0 0 0"/>
+            <geometry>
+                <box size="0.05 0.05 0.05" />
+            </geometry>
+            <material name="green" />
+        </visual>
+        <inertial>
+            <mass value="0.000001" />
+            <origin xyz="0 0 0" />
+            <inertia ixx="0.0001" ixy="0.0" ixz="0.0" iyy="0.0001" iyz="0.0" izz="0.0001" />
+        </inertial>
+    </link>
+    <joint name="laser" type="fixed">
+        <origin xyz="${chassisLength/2} 0 ${chassisHeight+0.001}" rpy="0 0 0" />
+        <parent link="chassis" />
+        <child link="base_laser_link" />
+    </joint>
 </robot>
