Commit message: Added maps and laser merger package

File: mybot_description/urdf/mybot.xacro (robot description, xacro)
@@ -68,9 +68,9 @@
     </link>
     <joint name="camera_joint" type="fixed">
-        <origin xyz="${chassisLength/2} 0 ${chassisHeight}" rpy="0.0 0.0 0.0"/>
+        <origin xyz="${chassisLength/2} 0.0 ${chassisHeight}" rpy="0.0 0.0 0.0"/>
         <parent link="chassis"/>
         <child link="camera"/>
     </joint>
-    <link name="base_laser_link">
+    <link name="base_laser_link_front">
         <visual>
             <origin xyz="0 0 0" rpy="0 0 0"/>
@@ -86,8 +86,27 @@
         </inertial>
     </link>
-    <joint name="laser" type="fixed">
+    <joint name="laser1" type="fixed">
         <origin xyz="${chassisLength/2} 0 ${chassisHeight+0.001}" rpy="0 0 0" />
         <parent link="chassis" />
-        <child link="base_laser_link" />
+        <child link="base_laser_link_front" />
+    </joint>
+     <link name="base_laser_link_rear">
+        <visual>
+            <origin xyz="0 0 0" rpy="0 0 0"/>
+            <geometry>
+                <box size="0.05 0.05 0.05" />
+            </geometry>
+            <material name="green" />
+        </visual>
+        <inertial>
+            <mass value="0.000001" />
+            <origin xyz="0 0 0" />
+            <inertia ixx="0.0001" ixy="0.0" ixz="0.0" iyy="0.0001" iyz="0.0" izz="0.0001" />
+        </inertial>
+    </link>
+    <joint name="laser2" type="fixed">
+        <origin xyz="-${chassisLength/2} 0 ${chassisHeight+0.001}" rpy="0 0 ${PI}" />
+        <parent link="chassis" />
+        <child link="base_laser_link_rear" />
     </joint>
 </robot>
