Commit message: added teb planner. Need to tweak the nav goal system

File: furbot_description/urdf/furbot.xacro (robot description, xacro)
@@ -40,4 +40,5 @@
     <link name="footprint" />
     <joint name="base_joint" type="fixed">
+        <origin xyz="${-chassisLength/2 + wheelPos} 0.0 ${wheelRadius}" rpy="0.0 0.0 0.0"/>
         <parent link="footprint"/>
         <child link="chassis"/>

File: furbot_description/urdf/macros.xacro (robot description, xacro)
@@ -102,5 +102,5 @@
             <child link="${lr}_steer"/>
             <axis xyz="0 0 1"/>
-            <limit lower="-1" upper="1" effort="100" velocity="100"/>
+            <limit lower="-2" upper="2" effort="100" velocity="100"/>
         </joint>>
         <joint name="${lr}_front_wheel_hinge" type="continuous">

Commit message: Dimensions modified. Pareters set up properly

File: furbot_description/urdf/furbot.xacro (robot description, xacro)
@@ -4,12 +4,12 @@
     <xacro:property name="PI" value="3.1415926535897931"/>
     <xacro:property name="chassisHeight" value="0.1"/>
-    <xacro:property name="chassisLength" value="0.6"/>
-    <xacro:property name="chassisWidth" value="0.2"/>
+    <xacro:property name="chassisLength" value="0.8"/>
+    <xacro:property name="chassisWidth" value="0.3"/>
     <xacro:property name="chassisMass" value="50"/>
     <xacro:property name="casterRadius" value="0.05"/>
     <xacro:property name="casterMass" value="5"/>
-    <xacro:property name="wheelWidth" value="0.05"/>
-    <xacro:property name="wheelRadius" value="0.08"/>
-    <xacro:property name="wheelPos" value="0.45"/>
+    <xacro:property name="wheelWidth" value="0.08"/>
+    <xacro:property name="wheelRadius" value="0.09"/>
+    <xacro:property name="wheelPos" value="0.65"/>
     <xacro:property name="wheelMass" value="5"/>
     <xacro:property name="cameraSize" value="0.05"/>
@@ -48,5 +48,5 @@
     <front_wheel lr="right" tY="-1" />
     <front_wheel lr="left" tY="1" />
-    <link name="camera">
+    <link name="furbot_camera">
         <collision>
             <origin xyz="0 0 0" rpy="0 0 0"/>
@@ -71,5 +71,5 @@
         <origin xyz="${chassisLength/2} 0.0 ${chassisHeight}" rpy="0.0 0.0 0.0"/>
         <parent link="chassis"/>
-        <child link="camera"/>
+        <child link="furbot_camera"/>
     </joint>
     <link name="base_laser_link_front">
@@ -88,5 +88,5 @@
     </link>
     <joint name="laser1" type="fixed">
-        <origin xyz="${chassisLength/2} 0 ${chassisHeight+0.001}" rpy="0 0 0" />
+        <origin xyz="${chassisLength/2 + 0.001} 0 ${chassisHeight+0.001}" rpy="0 0 0" />
         <parent link="chassis" />
         <child link="base_laser_link_front" />
@@ -107,5 +107,5 @@
     </link>
     <joint name="laser2" type="fixed">
-        <origin xyz="-${chassisLength/2} 0 ${chassisHeight+0.001}" rpy="0 0 ${PI}" />
+        <origin xyz="-${chassisLength/2 - 0.001} 0 ${chassisHeight+0.001}" rpy="0 0 ${PI}" />
         <parent link="chassis" />
         <child link="base_laser_link_rear" />

Commit message: Parameters and dimensions  correction

File: furbot_description/urdf/furbot.xacro (robot description, xacro)
@@ -3,5 +3,5 @@
     xmlns:xacro="http://www.ros.org/wiki/xacro">
     <xacro:property name="PI" value="3.1415926535897931"/>
-    <xacro:property name="chassisHeight" value="0.1"/>
+    <xacro:property name="chassisHeight" value="0.3"/>
     <xacro:property name="chassisLength" value="0.8"/>
     <xacro:property name="chassisWidth" value="0.3"/>
@@ -20,5 +20,5 @@
     <link name='chassis'>
         <collision>
-            <origin xyz="0 0 ${wheelRadius}" rpy="0 0 0"/>
+            <origin xyz="0 0 ${wheelRadius + chassisHeight/2}" rpy="0 0 0"/>
             <geometry>
                 <box size="${chassisLength} ${chassisWidth} ${chassisHeight}"/>
@@ -26,5 +26,5 @@
         </collision>
         <visual>
-            <origin xyz="0 0 ${wheelRadius}" rpy="0 0 0"/>
+            <origin xyz="0 0 ${wheelRadius + chassisHeight/2}" rpy="0 0 0"/>
             <geometry>
                 <box size="${chassisLength} ${chassisWidth} ${chassisHeight}"/>
@@ -33,5 +33,5 @@
         </visual>
         <inertial>
-            <origin xyz="0 0 ${wheelRadius}" rpy="0 0 0"/>
+            <origin xyz="0 0 ${wheelRadius + chassisHeight/2}" rpy="0 0 0"/>
             <mass value="${chassisMass}"/>
             <box_inertia m="${chassisMass}" x="${chassisLength}" y="${chassisWidth}" z="${chassisHeight}"/>
@@ -40,5 +40,5 @@
     <link name="footprint" />
     <joint name="base_joint" type="fixed">
-        <origin xyz="${-chassisLength/2 + wheelPos} 0.0 ${wheelRadius}" rpy="0.0 0.0 0.0"/>
+        <origin xyz="${-chassisLength/2 + wheelPos} 0.0 0" rpy="0.0 0.0 0.0"/>
         <parent link="footprint"/>
         <child link="chassis"/>
@@ -87,6 +87,6 @@
         </inertial>
     </link>
-    <joint name="laser1" type="fixed">
-        <origin xyz="${chassisLength/2 + 0.001} 0 ${chassisHeight+0.001}" rpy="0 0 0" />
+    <joint name="laser1" type="fixed">4
+        <origin xyz="${chassisLength/2 + 0.001} ${chassisWidth/2 + 0.001} ${wheelRadius*2 + 0.08}" rpy="0 0 0" />
         <parent link="chassis" />
         <child link="base_laser_link_front" />
@@ -107,5 +107,5 @@
     </link>
     <joint name="laser2" type="fixed">
-        <origin xyz="-${chassisLength/2 - 0.001} 0 ${chassisHeight+0.001}" rpy="0 0 ${PI}" />
+        <origin xyz="-${chassisLength/2 - 0.001} ${-chassisWidth/2 -0.001}  ${wheelRadius*2 + 0.08}" rpy="0 0 ${PI}" />
         <parent link="chassis" />
         <child link="base_laser_link_rear" />

File: furbot_description/urdf/materials.xacro (robot description, xacro)
@@ -21,5 +21,5 @@
     </material>
     <material name="red">
-        <color rgba="0.8 0.0 0.0 1.0"/>
+        <color rgba="0.79 0.17 0.0 1.0"/>
     </material>
     <material name="white">

Commit message: Furbot optimizations. New map

File: furbot_description/urdf/furbot.xacro (robot description, xacro)
@@ -87,6 +87,6 @@
         </inertial>
     </link>
-    <joint name="laser1" type="fixed">4
-        <origin xyz="${chassisLength/2 + 0.001} ${chassisWidth/2 + 0.001} ${wheelRadius*2 + 0.08}" rpy="0 0 0" />
+    <joint name="laser1" type="fixed">
+        <origin xyz="${chassisLength/2 + 0.001} ${-chassisWidth/2 - 0.001} ${wheelRadius*2 + 0.08}" rpy="0 0 0" />
         <parent link="chassis" />
         <child link="base_laser_link_front" />
@@ -94,5 +94,5 @@
      <link name="base_laser_link_rear">
         <visual>
-            <origin xyz="0 0 0" rpy="0 0 0"/>
+            <origin xyz="0 0 0" rpy="0 0 ${PI}"/>
             <geometry>
                 <box size="0.05 0.05 0.05" />
@@ -107,5 +107,5 @@
     </link>
     <joint name="laser2" type="fixed">
-        <origin xyz="-${chassisLength/2 - 0.001} ${-chassisWidth/2 -0.001}  ${wheelRadius*2 + 0.08}" rpy="0 0 ${PI}" />
+        <origin xyz="-${chassisLength/2 - 0.001} ${chassisWidth/2 +0.001}  ${wheelRadius*2 + 0.08}" rpy="0 0 ${PI}" />
         <parent link="chassis" />
         <child link="base_laser_link_rear" />
